File: 18650_Plugger_v1/18650_Plugger_v1.kicad_sch (KiCad schematic)
At the start: 1 part

Commit message: Schematic and PCB
Parts:
- added C1: 2µ2, Capacitor_SMD:C_0805_2012Metric, symbol Device:C_Small
- added C2, C3: 100n, Capacitor_SMD:C_0805_2012Metric, symbol Device:C_Small
- added D1: Red, LED_SMD:LED_0805_2012Metric, symbol Device:LED_Small
- added F1: 5A, Fuse:Fuse_0805_2012Metric, symbol Device:Fuse_Small
- added J1: USB_C_Receptacle_USB2.0, 18650_Plugger:GCT_USB4085-GF-A, symbol Connector:USB_C_Receptacle_USB2.0
- added J2, J3, J4, J5: Conn_01x12, 18650_Plugger:PinHeader_1x12_P2.54mm_Vertical, symbol Connector_Generic:Conn_01x12
- added R1, R2: 5k1, Resistor_SMD:R_0805_2012Metric, symbol Device:R_Small
- added R3, R6: 330, Resistor_SMD:R_0805_2012Metric, symbol Device:R_Small
- added R4: 432, Resistor_SMD:R_0805_2012Metric, symbol Device:R_Small
- added R5: 1k05, Resistor_SMD:R_0805_2012Metric, symbol Device:R_Small
- added R7: 2k2, Resistor_SMD:R_0805_2012Metric, symbol Device:R_Small
- added U1: TPS2113APWR, Package_SO:TSSOP-8_4.4x3mm_P0.65mm, symbol 18650_Plugger:TPS2113APWR
- added U2: MCP73113-16SI/MF, Package_DFN_QFN:DFN-10-1EP_3x3mm_P0.5mm_EP1.55x2.48mm, symbol 18650_Plugger:MCP73113-16SI/MF
- added U3: AP9214LA-AH-HSB-7, 18650_Plugger:U-DFN2535-6 (Type B), symbol 18650_Plugger:AP9214LA-AH-HSB-7
- BT1: renamed from BT?; footprint (none) -> 18650_Plugger:Keystone_254_holder
Connections:
- net +BATT: now reaches BT1.1 (+)
- net +BATT: now also F1.1
- net -BATT: now reaches BT1.2 (-)
- net -BATT: now also C3.2, U3.1 (S1), U3.2 (VSS)
- new net: R4.1, U1.4 (ILIM)
- new net: J1.B5 (CC2), R1.1
- new net: R5.1, U2.10 (PROG)
- new net: J1.A5 (CC1), R2.1
- new net: C3.1, R6.1, U3.3 (VDD)
- new net: R7.1, U3.4 (VM)
- new net: D1.1 (K), R3.1
- new net GND: C1.2, C2.2, J1.A1 (GND), J1.A12 (GND), J1.B1 (GND), J1.B12 (GND), J4.1 (Pin_1), J4.10 (Pin_10), J4.11 (Pin_11), J4.12 (Pin_12), J4.2 (Pin_2), J4.3 (Pin_3), J4.4 (Pin_4), J4.5 (Pin_5), J4.6 (Pin_6), J4.7 (Pin_7), J4.8 (Pin_8), J4.9 (Pin_9), J5.1 (Pin_1), J5.10 (Pin_10), J5.11 (Pin_11), J5.12 (Pin_12), J5.2 (Pin_2), J5.3 (Pin_3), J5.4 (Pin_4), J5.5 (Pin_5), J5.6 (Pin_6), J5.7 (Pin_7), J5.8 (Pin_8), J5.9 (Pin_9), R1.2, R2.2, R4.2, R5.2, R7.2, U1.2 (~EN), U1.3 (VSNS), U1.5 (GND), U2.11 (EP), U2.8 (VSS), U2.9 (VSS), U3.6 (S2)
- new net P+: F1.2, R6.2, U1.6 (IN2), U2.3 (VBAT), U2.4 (VBAT)
- new net STAT: R3.2, U2.7 (STAT)
- new net VBUS: D1.2 (A), J1.A4 (VBUS), J1.A9 (VBUS), J1.B4 (VBUS), J1.B9 (VBUS), U1.8 (IN1), U2.1 (VDD), U2.2 (VDD)
- new net VDD: C1.1, C2.1, J2.1 (Pin_1), J2.10 (Pin_10), J2.11 (Pin_11), J2.12 (Pin_12), J2.2 (Pin_2), J2.3 (Pin_3), J2.4 (Pin_4), J2.5 (Pin_5), J2.6 (Pin_6), J2.7 (Pin_7), J2.8 (Pin_8), J2.9 (Pin_9), J3.1 (Pin_1), J3.10 (Pin_10), J3.11 (Pin_11), J3.12 (Pin_12), J3.2 (Pin_2), J3.3 (Pin_3), J3.4 (Pin_4), J3.5 (Pin_5), J3.6 (Pin_6), J3.7 (Pin_7), J3.8 (Pin_8), J3.9 (Pin_9), U1.7 (OUT)
- no-connect marks 0 -> 9
Other:
- note added: "BMS for a single Li-ion cell. Recommended charging voltage: 5V Maximum output current: 1.15A, limited by the OR-controller."
- note added: "Charging circuit"
- note added: "Connectors"
- note added: "DC-input"
- note added: "I_CHG = 1104*R_PROG^(-0.93) R_PROG = 1.05kΩ -> I_CHG = 1.055A"
- note added: "I_LIM = 500/R_LIM R_LIM = 432Ω -> I_LIM = 1.15A"
- note added: "LED indicator: ON = charging OFF = done charging"
- note added: "OR-controller"
- note added: "Protection circuit"
- note added: "Typ. quiescent current is 3µA in normal mode"
- note added: "Typ. quiescent current while operating is 55µA, but if ~EN is high, standby quiesc. curr. is typ 0.5µA"
- moved on the sheet: BT1
